File: WallSwitch/WallSwitch.sch (EAGLE design)
At the start: 37 parts, among them IC1 WS2811, IC2 AT42QT1010-TSHR, IC3 LNK306DG, IC4 WS2811, IC5 AT42QT1010-TSHR, IC6 AP2112K-3.3TRG1, J1 AC Line, J2 Interface

Commit message: foo
Parts:
- removed L1: 1mH, freetronics-luke:INDUCTOR2MM
- removed L2: 680µH, freetronics-luke:INDUCTOR5MM
- added L3: 1mH, freetronics-luke:LRLB0608
- added L4: 680µH, freetronics-luke:LRLB0914
- C1, C7: value 2.2nF -> 4.7nF
Connections:
- removed net N$8: D1.A, R3.2
- new net N$7: D1.A, R3.1
- net +4V: now also L4.2; no longer L2.2
- net N$10: now also L3.2; no longer L1.2
- net N$12: now also L4.1; no longer L2.1
- net N$2: now also R3.2; no longer R3.1
- net N$9: now also L3.1; no longer L1.1
Other:
- moved on the sheet: R3
