File: PowerNode/PowerNode.sch (EAGLE design)
At the start: 43 parts, among them IC1 AP2112K-3.3TRG1, IC2 ATM90E26-YU-B, IC3 LNK306DG, J1 AC Load, J2 AC Line, J3 Interface, Q1 8.192MHz, Q2 2N7002

Commit message: foo
Parts:
- L1: device freetronics-luke:INDUCTOR2MM -> freetronics-luke:LRLB0608
- L2: device freetronics-luke:INDUCTOR5MM -> freetronics-luke:LRLB0914
Connections:
- net N$4 renamed GND
Other:
- moved on the sheet: C11, D1, R8
Changed lines of the file:
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@@
 <attribute name="VOLTAGE" value="400V"/>
 </part>
-<part name="L2" library="freetronics-luke" deviceset="INDUCTOR" device="5MM" value="680µH"/>
 <part name="R8" library="freetronics-luke" deviceset="RESISTOR" device="FKN200JR-73" value="8.2Ω">
 <attribute name="FOO" value="Fusible"/>
@@
 <attribute name="PACKAGE" value="7-SOIC"/>
 </part>
-<part name="L1" library="freetronics-luke" deviceset="INDUCTOR" device="2MM" value="1mH"/>
 <part name="C12" library="freetronics-luke" deviceset="ELECTROLYTIC" device="3.5MM" value="4.7µF">
 <attribute name="VOLTAGE" value="400V"/>
@@
 </part>
 <part name="U$2" library="freetronics-luke" deviceset="GND" device=""/>
+<part name="L1" library="freetronics-luke" deviceset="L" device="RLB0608" value="1mH"/>
+<part name="L2" library="freetronics-luke" deviceset="L" device="RLB0914" value="680µH"/>
 </parts>
 <sheets>
@@
 <attribute name="VALUE" x="231.14" y="50.8" size="1.27" layer="96"/>
 </instance>
-<instance part="C11" gate="G$1" x="144.78" y="50.8" smashed="yes">
-<attribute name="VOLTAGE" x="137.16" y="48.26" size="1.27" layer="96"/>
-<attribute name="NAME" x="137.16" y="53.34" size="1.27" layer="95"/>
-<attribute name="VALUE" x="137.16" y="50.8" size="1.27" layer="96"/>
-</instance>
-<instance part="L2" gate="G$1" x="226.06" y="58.42" smashed="yes">
-<attribute name="NAME" x="220.98" y="55.88" size="1.27" layer="95"/>
-<attribute name="VALUE" x="220.98" y="53.34" size="1.27" layer="96"/>
-</instance>
-<instance part="R8" gate="G$1" x="130.81" y="58.42" smashed="yes">
-<attribute name="ID" x="116.84" y="63.5" size="1.27" layer="96"/>
-<attribute name="FOO" x="116.84" y="66.04" size="1.27" layer="96"/>
-<attribute name="POWER" x="121.92" y="68.58" size="1.27" layer="96"/>
-<attribute name="NAME" x="116.84" y="71.12" size="1.27" layer="95"/>
-<attribute name="VALUE" x="116.84" y="68.58" size="1.27" layer="96"/>
+<instance part="C11" gate="G$1" x="149.86" y="50.8" smashed="yes">
+<attribute name="VOLTAGE" x="142.24" y="48.26" size="1.27" layer="96"/>
+<attribute name="NAME" x="142.24" y="53.34" size="1.27" layer="95"/>
+<attribute name="VALUE" x="142.24" y="50.8" size="1.27" layer="96"/>
+</instance>
+<instance part="R8" gate="G$1" x="135.89" y="58.42" smashed="yes">
+<attribute name="ID" x="121.92" y="63.5" size="1.27" layer="96"/>
+<attribute name="FOO" x="121.92" y="66.04" size="1.27" layer="96"/>
+<attribute name="POWER" x="127" y="68.58" size="1.27" layer="96"/>
+<attribute name="NAME" x="121.92" y="71.12" size="1.27" layer="95"/>
+<attribute name="VALUE" x="121.92" y="68.58" size="1.27" layer="96"/>
 </instance>
 <instance part="IC3" gate="G$1" x="177.8" y="55.88" smashed="yes">
@@
 <attribute name="VALUE" x="180.34" y="68.58" size="1.27" layer="96"/>
 </instance>
-<instance part="L1" gate="G$1" x="154.94" y="58.42" smashed="yes">
-<attribute name="NAME" x="149.86" y="63.5" size="1.27" layer="95"/>
-<attribute name="VALUE" x="149.86" y="60.96" size="1.27" layer="96"/>
-</instance>
 <instance part="C12" gate="G$1" x="165.1" y="50.8" smashed="yes">
 <attribute name="VOLTAGE" x="157.48" y="48.26" size="1.27" layer="96"/>
@@
 <attribute name="VALUE" x="157.48" y="50.8" size="1.27" layer="96"/>
 </instance>
-<instance part="U$9" gate="G$1" x="144.78" y="43.18"/>
+<instance part="U$9" gate="G$1" x="149.86" y="43.18"/>
 <instance part="U$10" gate="G$1" x="165.1" y="43.18"/>
 <instance part="U$11" gate="G$1" x="215.9" y="43.18"/>
@@
 </instance>
 <instance part="U$1" gate="G$1" x="71.12" y="106.68"/>
-<instance part="D1" gate="G$1" x="139.7" y="58.42" smashed="yes" rot="MR180">
-<attribute name="NAME" x="137.16" y="68.58" size="1.27" layer="95"/>
-<attribute name="VALUE" x="137.16" y="66.04" size="1.27" layer="96"/>
-<attribute name="PACKAGE" x="137.16" y="63.5" size="1.27" layer="96"/>
+<instance part="D1" gate="G$1" x="144.78" y="58.42" smashed="yes" rot="MR180">
+<attribute name="NAME" x="142.24" y="68.58" size="1.27" layer="95"/>
+<attribute name="VALUE" x="142.24" y="66.04" size="1.27" layer="96"/>
+<attribute name="PACKAGE" x="142.24" y="63.5" size="1.27" layer="96"/>
 </instance>
 <instance part="D2" gate="G$1" x="215.9" y="50.8" smashed="yes" rot="MR90">
@@
 </instance>
 <instance part="U$2" gate="G$1" x="63.5" y="15.24" rot="MR0"/>
+<instance part="L1" gate="G$1" x="157.48" y="58.42" smashed="yes">
+<attribute name="NAME" x="152.4" y="63.5" size="1.27" layer="95"/>
+<attribute name="VALUE" x="152.4" y="60.96" size="1.27" layer="96"/>
+</instance>
+<instance part="L2" gate="G$1" x="226.06" y="58.42" smashed="yes">
+<attribute name="NAME" x="220.98" y="55.88" size="1.27" layer="95"/>
+<attribute name="VALUE" x="220.98" y="53.34" size="1.27" layer="96"/>
+</instance>
 </instances>
 <busses>
@@
 <net name="N$8" class="0">
 <segment>
-<wire x1="137.16" y1="58.42" x2="134.62" y2="58.42" width="0.1524" layer="91"/>
+<wire x1="142.24" y1="58.42" x2="139.7" y2="58.42" width="0.1524" layer="91"/>
 <pinref part="R8" gate="G$1" pin="2"/>
 <pinref part="D1" gate="G$1" pin="A"/>
@@
 <net name="N$9" class="0">
 <segment>
+<wire x1="152.4" y1="58.42" x2="149.86" y2="58.42" width="0.1524" layer="91"/>
+<pinref part="C11" gate="G$1" pin="+"/>
+<wire x1="149.86" y1="58.42" x2="147.32" y2="58.42" width="0.1524" layer="91"/>
+<wire x1="149.86" y1="55.88" x2="149.86" y2="58.42" width="0.1524" layer="91"/>
+<junction x="149.86" y="58.42"/>
+<pinref part="D1" gate="G$1" pin="K"/>
 <pinref part="L1" gate="G$1" pin="1"/>
-<wire x1="147.32" y1="58.42" x2="144.78" y2="58.42" width="0.1524" layer="91"/>
-<pinref part="C11" gate="G$1" pin="+"/>
-<wire x1="144.78" y1="58.42" x2="142.24" y2="58.42" width="0.1524" layer="91"/>
-<wire x1="144.78" y1="55.88" x2="144.78" y2="58.42" width="0.1524" layer="91"/>
-<junction x="144.78" y="58.42"/>
-<pinref part="D1" gate="G$1" pin="K"/>
 </segment>
 </net>
 <net name="N$10" class="0">
 <segment>
-<pinref part="L1" gate="G$1" pin="2"/>
 <pinref part="IC3" gate="G$1" pin="D"/>
 <wire x1="167.64" y1="58.42" x2="165.1" y2="58.42" width="0.1524" layer="91"/>
@@
 <wire x1="165.1" y1="55.88" x2="165.1" y2="58.42" width="0.1524" layer="91"/>
 <junction x="165.1" y="58.42"/>
+<pinref part="L1" gate="G$1" pin="2"/>
 </segment>
 </net>
@@
 <wire x1="200.66" y1="60.96" x2="200.66" y2="58.42" width="0.1524" layer="91"/>
 <pinref part="C16" gate="G$1" pin="1"/>
-<pinref part="L2" gate="G$1" pin="1"/>
 <junction x="200.66" y="58.42"/>
 <junction x="215.9" y="58.42"/>
 <wire x1="215.9" y1="53.34" x2="215.9" y2="58.42" width="0.1524" layer="91"/>
-<wire x1="218.44" y1="58.42" x2="215.9" y2="58.42" width="0.1524" layer="91"/>
+<wire x1="220.98" y1="58.42" x2="215.9" y2="58.42" width="0.1524" layer="91"/>
 <wire x1="215.9" y1="60.96" x2="215.9" y2="58.42" width="0.1524" layer="91"/>
 <wire x1="215.9" y1="58.42" x2="200.66" y2="58.42" width="0.1524" layer="91"/>
@@
 <pinref part="R9" gate="G$1" pin="1"/>
 <pinref part="D2" gate="G$1" pin="K"/>
+<pinref part="L2" gate="G$1" pin="1"/>
 </segment>
 </net>
@@
 <segment>
 <pinref part="R8" gate="G$1" pin="1"/>
-<wire x1="124.46" y1="58.42" x2="121.92" y2="58.42" width="0.1524" layer="91"/>
-<label x="121.92" y="58.42" size="1.27" layer="95" rot="R180" xref="yes"/>
+<wire x1="129.54" y1="58.42" x2="127" y2="58.42" width="0.1524" layer="91"/>
+<label x="127" y="58.42" size="1.27" layer="95" rot="R180" xref="yes"/>
 </segment>
 <segment>
@@
 </segment>
 </net>
-<net name="N$4" class="0">
+<net name="GND" class="0">
 <segment>
 <pinref part="U$48" gate="G$1" pin="GND"/>
@@
 <pinref part="C11" gate="G$1" pin="-"/>
 <pinref part="U$9" gate="G$1" pin="GND"/>
-<wire x1="144.78" y1="45.72" x2="144.78" y2="48.26" width="0.1524" layer="91"/>
+<wire x1="149.86" y1="45.72" x2="149.86" y2="48.26" width="0.1524" layer="91"/>
 </segment>
 <segment>
@@
 </segment>
 <segment>
-<pinref part="L2" gate="G$1" pin="2"/>
-<wire x1="233.68" y1="58.42" x2="241.3" y2="58.42" width="0.1524" layer="91"/>
+<wire x1="231.14" y1="58.42" x2="241.3" y2="58.42" width="0.1524" layer="91"/>
 <wire x1="241.3" y1="58.42" x2="241.3" y2="63.5" width="0.1524" layer="91"/>
 <pinref part="C17" gate="G$1" pin="+"/>
@@
 <pinref part="U$41" gate="G$1" pin="+5V"/>
 <pinref part="D4" gate="G$1" pin="A"/>
-</segment>
-<segment>
+<pinref part="L2" gate="G$1" pin="2"/>
+</segment>
+<segment>
