File: PowerNode/PowerNode.brd (EAGLE design)
At the start: 60 x 34.4 mm, 43 parts, among them IC1 AP2112K-3.3TRG1, IC2 ATM90E26-YU-B, IC3 LNK306DG, J1 AC Load, J2 AC Line, J3 Interface, Q1 8.192MHz, Q2 2N7002

Commit message: foo
Parts:
- L1: device freetronics-luke:INDUCTOR_SMALL -> freetronics-luke:RLB0608
- L2: device freetronics-luke:INDUCTOR-LARGE -> freetronics-luke:RLB0914
- moved D4 0.45 mm to (10.2, 26.4)
Connections:
- net N$4 renamed GND
Routing:
- net +3.3V: track 38.0 -> 39.3 mm
- net N$16: track 11.3 -> 10.3 mm
- net +4V: track 42.4 -> 43.0 mm
Changed lines of the file:
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@@
 <layer number="21" name="tPlace" color="7" fill="1" visible="yes" active="yes"/>
 <layer number="22" name="bPlace" color="11" fill="1" visible="yes" active="yes"/>
-<layer number="23" name="tOrigins" color="15" fill="1" visible="no" active="yes"/>
+<layer number="23" name="tOrigins" color="15" fill="1" visible="yes" active="yes"/>
 <layer number="24" name="bOrigins" color="15" fill="1" visible="no" active="yes"/>
 <layer number="25" name="tNames" color="7" fill="1" visible="no" active="yes"/>
@@
 <attribute name="VALUE" x="2.8575" y="2.54" size="0.8128" layer="27" ratio="15"/>
 </element>
-<element name="L2" library="freetronics-luke" package="INDUCTOR-LARGE" value="680µH" x="4.1275" y="29.845" smashed="yes">
-<attribute name="NAME" x="0.635" y="25.4" size="0.8128" layer="25" font="vector" ratio="15"/>
-<attribute name="VALUE" x="2.2225" y="27.6225" size="0.8128" layer="27" font="vector" ratio="15"/>
-</element>
 <element name="R8" library="freetronics-luke" package="FKN200JR-73" value="8.2Ω" x="16.51" y="11.43" smashed="yes" rot="R90">
 <attribute name="ID" value="FKN200JR-73-8R2" x="16.51" y="11.43" size="1.778" layer="27" rot="R90" display="off"/>
@@
 <attribute name="VALUE" x="2.2225" y="20.955" size="0.8128" layer="27" ratio="15"/>
 <attribute name="NAME" x="0.635" y="17.4625" size="0.8128" layer="25" ratio="15"/>
-</element>
-<element name="L1" library="freetronics-luke" package="INDUCTOR_SMALL" value="1mH" x="11.1125" y="11.43" smashed="yes" rot="R180">
-<attribute name="NAME" x="7.3025" y="9.2075" size="0.8128" layer="25" font="vector" ratio="15"/>
-<attribute name="VALUE" x="9.8425" y="9.525" size="0.8128" layer="27" font="vector" ratio="15"/>
 </element>
 <element name="C12" library="freetronics-luke" package="ELECTRO-LARGE" value="4.7µF" x="4.445" y="13.335" smashed="yes" rot="R180">
@@
 <attribute name="VALUE" x="13.6525" y="26.3525" size="0.8128" layer="27" ratio="15"/>
 </element>
-<element name="D4" library="freetronics-luke" package="SMA" value="S1J-13-F" x="9.8425" y="26.67" smashed="yes" rot="R270">
-<attribute name="PACKAGE" value="SMA" x="9.8425" y="26.67" size="1.778" layer="27" rot="R270" display="off"/>
-<attribute name="NAME" x="11.7475" y="26.3525" size="0.8128" layer="25" ratio="15"/>
-<attribute name="VALUE" x="10.16" y="23.8125" size="0.8128" layer="27" ratio="15" rot="R90"/>
-</element>
+<element name="D4" library="freetronics-luke" package="SMA" value="S1J-13-F" x="10.16" y="26.3525" smashed="yes" rot="R270">
+<attribute name="PACKAGE" value="SMA" x="10.16" y="26.3525" size="1.778" layer="27" rot="R270" display="off"/>
+<attribute name="NAME" x="12.065" y="26.035" size="0.8128" layer="25" ratio="15"/>
+<attribute name="VALUE" x="10.4775" y="23.495" size="0.8128" layer="27" ratio="15" rot="R90"/>
+</element>
+<element name="L1" library="freetronics-luke" package="RLB0608" value="1mH" x="11.1125" y="11.43" rot="R180"/>
+<element name="L2" library="freetronics-luke" package="RLB0914" value="680µH" x="4.1275" y="29.845"/>
 </elements>
 <signals>
@@
 </signal>
 <signal name="N$9">
-<contactref element="L1" pad="1"/>
 <contactref element="C11" pad="+"/>
 <contactref element="D1" pad="K"/>
-<wire x1="12.1125" y1="11.43" x2="12.1125" y2="10.3625" width="1.016" layer="1"/>
-<wire x1="12.1125" y1="10.3625" x2="6.195" y2="4.445" width="1.016" layer="1"/>
 <wire x1="9.915" y1="15.875" x2="9.915" y2="14.69125" width="1.143" layer="1"/>
 <wire x1="9.915" y1="14.69125" x2="12.1125" y2="12.49375" width="1.143" layer="1"/>
-<wire x1="12.1125" y1="11.43" x2="12.1125" y2="12.49375" width="1.143" layer="1"/>
+<contactref element="L1" pad="1"/>
+<wire x1="12.1125" y1="11.43" x2="12.1125" y2="10.3625" width="1.143" layer="1"/>
+<wire x1="12.1125" y1="10.3625" x2="6.195" y2="4.445" width="1.143" layer="1"/>
+<wire x1="12.1125" y1="12.49375" x2="12.1125" y2="11.43" width="1.143" layer="1"/>
 </signal>
 <signal name="N$10">
-<contactref element="L1" pad="2"/>
 <contactref element="IC3" pad="4"/>
 <contactref element="C12" pad="+"/>
 <wire x1="7.14375" y1="18.9738" x2="7.14375" y2="16.35125" width="0.508" layer="1"/>
 <wire x1="7.14375" y1="16.35125" x2="6.195" y2="15.4025" width="0.508" layer="1"/>
-<wire x1="10.1125" y1="11.43" x2="8.1" y2="11.43" width="1.524" layer="16"/>
-<wire x1="8.1" y1="11.43" x2="6.195" y2="13.335" width="1.524" layer="16"/>
+<wire x1="8.1" y1="11.43" x2="7.86" y2="11.67" width="1.524" layer="16"/>
+<wire x1="7.86" y1="11.67" x2="6.195" y2="13.335" width="1.524" layer="16"/>
 <wire x1="6.195" y1="13.335" x2="6.195" y2="15.4025" width="0.508" layer="1"/>
+<contactref element="L1" pad="2"/>
+<wire x1="10.1125" y1="11.43" x2="8.1" y2="11.43" width="1.143" layer="16"/>
 </signal>
 <signal name="N$11">
@@
 <contactref element="IC3" pad="7"/>
 <contactref element="C16" pad="1"/>
-<contactref element="L2" pad="1"/>
 <contactref element="C14" pad="2"/>
 <contactref element="R9" pad="1"/>
@@
 <vertex x="-6" y="34.365"/>
 <vertex x="15.5575" y="34.365"/>
-<vertex x="15.5575" y="21.59"/>
-<vertex x="-6" y="21.59"/>
+<vertex x="15.5575" y="21.9075"/>
+<vertex x="-6" y="21.9075"/>
 </polygon>
+<contactref element="L2" pad="1"/>
 </signal>
 <signal name="N$15">
@@
 <contactref element="R10" pad="1"/>
 <contactref element="D4" pad="K"/>
-<wire x1="9.8425" y1="24.52" x2="12.22375" y2="24.52" width="0.4064" layer="1"/>
+<wire x1="10.16" y1="24.2025" x2="12.22375" y2="24.2025" width="0.4064" layer="1"/>
 <wire x1="14.44625" y1="20.69" x2="14.44625" y2="19.685" width="0.4064" layer="1"/>
 <via x="14.44625" y="19.685" extent="1-16" drill="0.3302"/>
-<via x="12.22375" y="24.52" extent="1-16" drill="0.3302"/>
-<wire x1="12.22375" y1="24.52" x2="12.22375" y2="22.39" width="0.4064" layer="1"/>
-<wire x1="12.22375" y1="24.52" x2="12.22375" y2="21.9075" width="0.4064" layer="16"/>
+<via x="12.22375" y="24.2025" extent="1-16" drill="0.3302"/>
+<wire x1="12.22375" y1="24.2025" x2="12.22375" y2="22.39" width="0.4064" layer="1"/>
+<wire x1="12.22375" y1="24.2025" x2="12.22375" y2="21.9075" width="0.4064" layer="16"/>
 <wire x1="12.22375" y1="21.9075" x2="14.44625" y2="19.685" width="0.4064" layer="16"/>
 </signal>
@@
 <wire x1="39.52875" y1="17.6275" x2="41.75125" y2="17.6275" width="0.4064" layer="16"/>
 <wire x1="38.985" y1="20.1565" x2="38.985" y2="24.515" width="0.3048" layer="1"/>
-<wire x1="38.985" y1="24.515" x2="37.685" y2="25.815" width="0.3048" layer="1"/>
 <wire x1="39.635" y1="20.1565" x2="39.635" y2="19.315" width="0.3048" layer="1"/>
 <wire x1="39.52875" y1="18.7325" x2="39.52875" y2="19.20875" width="0.3048" layer="1"/>
@@
 <via x="37.685" y="25.815" extent="1-16" drill="0.3302"/>
 <wire x1="37.685" y1="27.4685" x2="37.685" y2="25.815" width="0.3048" layer="1"/>
-<wire x1="21.7775" y1="29.5275" x2="33.9725" y2="29.5275" width="0.4064" layer="16"/>
-<wire x1="33.9725" y1="29.5275" x2="37.685" y2="25.815" width="0.4064" layer="16"/>
+<wire x1="21.7775" y1="29.5275" x2="36.195" y2="29.5275" width="0.4064" layer="16"/>
+<wire x1="36.195" y1="29.5275" x2="37.685" y2="28.0375" width="0.4064" layer="16"/>
+<wire x1="37.685" y1="25.815" x2="37.685" y2="28.0375" width="0.4064" layer="16"/>
+<wire x1="38.985" y1="24.515" x2="37.685" y2="25.815" width="0.3048" layer="1"/>
 </signal>
 <signal name="VREF">
@@
 <contactref element="IC1" pad="1"/>
 <contactref element="IC1" pad="3"/>
-<contactref element="L2" pad="2"/>
 <contactref element="C17" pad="+"/>
 <contactref element="D3" pad="1"/>
@@
 <contactref element="C1" pad="1"/>
 <contactref element="D4" pad="A"/>
-<wire x1="9.8425" y1="28.82" x2="9.8425" y2="30.36875" width="0.889" layer="1"/>
-<wire x1="9.8425" y1="30.36875" x2="11.22375" y2="31.75" width="0.889" layer="1"/>
+<wire x1="10.16" y1="28.5025" x2="10.16" y2="30.68625" width="0.889" layer="1"/>
+<wire x1="10.16" y1="30.68625" x2="11.22375" y2="31.75" width="0.889" layer="1"/>
 <wire x1="22.54" y1="24.7349" x2="23.1474" y2="24.7349" width="0.4064" layer="1"/>
 <wire x1="23.1474" y1="24.7349" x2="23.6475" y2="25.235" width="0.4064" layer="1"/>
 <wire x1="24.765" y1="25.235" x2="23.6475" y2="25.235" width="0.4064" layer="1"/>
-<wire x1="9.8425" y1="28.82" x2="7.6525" y2="28.82" width="0.889" layer="1"/>
-<wire x1="7.6525" y1="28.82" x2="6.6275" y2="29.845" width="0.889" layer="1"/>
 <wire x1="13.6525" y1="33.17875" x2="12.6525" y2="33.17875" width="0.4064" layer="16"/>
 <wire x1="12.6525" y1="33.17875" x2="11.22375" y2="31.75" width="0.4064" layer="16"/>
@@
 <wire x1="16.51" y1="30.32125" x2="16.51" y2="23.6925" width="0.4064" layer="16"/>
 <wire x1="16.51" y1="23.6925" x2="21.935" y2="18.2675" width="0.4064" layer="16"/>
+<contactref element="L2" pad="2"/>
+<wire x1="10.16" y1="28.5025" x2="7.97" y2="28.5025" width="1.143" layer="1"/>
+<wire x1="7.97" y1="28.5025" x2="6.6275" y2="29.845" width="1.143" layer="1"/>
 </signal>
 <signal name="N$2">
@@
 <wire x1="33.935" y1="10.8325" x2="33.935" y2="6.0675" width="2.54" layer="16"/>
 </signal>
-<signal name="N$4">
+<signal name="GND">
 <wire x1="17.4625" y1="2.2225" x2="17.145" y2="3.4925" width="0.8128" layer="16"/>
 <wire x1="19.3675" y1="2.2225" x2="19.685" y2="1.905" width="0.8128" layer="16"/>

Commit message: foo
Routing:
- net GND: track 243.8 -> 246.0 mm
